Commit message: add gripper in urdf

File: src/tm_description/urdf/tm5-900.urdf (robot description, URDF)
Before this commit: robot tm5-900, 10 links, 9 joints
Links:
- added link gripper; collision mesh filename=package://tm_description/meshes/Gripper.stl; visual mesh filename=package://tm_description/meshes/Gripper.stl
Joints:
- added joint gripper_joint: type fixed, parent link_6, child gripper, origin xyz=0.000000 0.000000 0.000000 rpy=0.000000 0.000000 0.000000

File: src/tm_description/xacro/macro.tm5-900-nominal.urdf.xacro (robot description, xacro)
@@ -280,4 +280,24 @@
     <origin rpy="0.000000 0.000000 0.000000" xyz="0.000000 0.000000 0.000000" />
   </joint>
+  <link name="gripper">
+    <visual>
+      <geometry>
+        <mesh scale="0.001 0.001 0.001" filename="package://tm_description/meshes/Assembly1.stl"/>
+      </geometry>
+      <material name="Grey">
+        <color rgba="0.9 0.9 0.9 1.0"/>
+      </material>
+    </visual>
+    <collision>
+      <geometry>
+        <mesh scale="0.001 0.001 0.001" filename="package://tm_description/meshes/Assembly1.stl"/>
+      </geometry>
+    </collision>
+  </link>
+  <joint name="gripper_joint" type="fixed">
+    <parent link="${prefix}link_6"/>
+    <child link="gripper"/>
+    <origin rpy="-1.570795 0.000000 -1.570795" xyz="0.0224 0.0001 0.1568"/>
+  </joint>
 <!--LinkDescription-->
   </xacro:macro>

Commit message: make arm scan the environment

File: src/tm_description/urdf/tm5-900.urdf (robot description, URDF)
Before this commit: robot tm5-900, 11 links, 10 joints
Links:
- link gripper: geometry collision mesh filename=package://tm_description/meshes/gripper2023v1.stl; visual mesh filename=package://tm_description/meshes/gripper2023v1.stl

Commit message: alter urdf/camera_broadcaster

File: src/tm_description/urdf/tm5-900.urdf (robot description, URDF)
Before this commit: robot tm5-900, 11 links, 10 joints
Links:
- added link camera
- link gripper: geometry collision mesh filename=package://tm_description/meshes/gripper2023v1.stl scale=0.001 0.001 0.001; visual mesh filename=package://tm_description/meshes/gripper2023v1.stl scale=0.001 0.001 0.001
Joints:
- added joint camera_joint: type fixed, parent ${prefix}link_6, child camera, origin xyz=-0.0585 -0.0115 0.15995 rpy=0.00000 0.000000 -1.570795
- joint gripper_joint: origin xyz=0.000000 0.000000 0.000000 rpy=0.000000 0.000000 0.000000 -> xyz=0 0 0.132 rpy=-1.570795 0.000000 -1.570795; parent link_6 -> ${prefix}link_6

File: src/tm_description/xacro/macro.tm5-900-nominal.urdf.xacro (robot description, xacro)
@@ -301,6 +301,5 @@
   </joint>
   <disable_collisions link1="gripper" link2="link_6" reason="Never" />
-  <link name="camera">
-  </link>
+  <link name="camera"/>
   <joint name="camera_joint" type="fixed">
     <parent link="${prefix}link_6"/>

File: src/tm_description/xacro/macro.tm5x-900-nominal.urdf.xacro (robot description, xacro)
@@ -280,4 +280,32 @@
     <origin rpy="0.000000 0.000000 0.000000" xyz="0.000000 0.000000 0.000000" />
   </joint>
+  <link name="gripper">
+    <visual>
+      <geometry>
+        <mesh scale="0.001 0.001 0.001" filename="package://tm_description/meshes/gripper2023v1.stl"/>
+      </geometry>
+      <material name="Grey">
+        <color rgba="0.9 0.9 0.9 1.0"/>
+      </material>
+    </visual>
+    <collision>
+      <geometry>
+        <mesh scale="0.001 0.001 0.001" filename="package://tm_description/meshes/gripper2023v1.stl"/>
+      </geometry>
+    </collision>
+  </link>
+  <joint name="gripper_joint" type="fixed">
+    <parent link="${prefix}link_6"/>
+    <child link="gripper"/>
+    <origin rpy="-1.570795 0.000000 -1.570795" xyz="0 0 0.132"/>
+  </joint>
+  <disable_collisions link1="gripper" link2="link_6" reason="Never" />
+  <link name="camera">
+  </link>
+  <joint name="camera_joint" type="fixed">
+    <parent link="${prefix}link_6"/>
+    <child link="camera"/>
+    <origin rpy="0.00000 0.000000 -1.570795" xyz="-0.0585 -0.0115 0.15995"/>
+  </joint>
 <!--LinkDescription-->
   </xacro:macro>

Commit message: Comment the gripper to resolve the collision problem

File: src/tm_description/urdf/tm5-900.urdf (robot description, URDF)
Before this commit: robot tm5-900, 12 links, 11 joints
Links:
- removed link gripper
Joints:
- removed joint gripper_joint

File: src/tm_description/xacro/macro.tm5-900-nominal.urdf.xacro (robot description, xacro)
@@ -280,5 +280,5 @@
     <origin rpy="0.000000 0.000000 0.000000" xyz="0.000000 0.000000 0.000000" />
   </joint>
-  <link name="gripper">
+  <!-- <link name="gripper">
     <visual>
       <geometry>
@@ -294,11 +294,11 @@
       </geometry>
     </collision>
-  </link>
-  <joint name="gripper_joint" type="fixed">
+  </link> -->
+  <!-- <joint name="gripper_joint" type="fixed">
     <parent link="${prefix}link_6"/>
     <child link="gripper"/>
     <origin rpy="-1.570795 0.000000 -1.570795" xyz="0 0 0.132"/>
-  </joint>
-  <disable_collisions link1="gripper" link2="link_6" reason="Never" />
+  </joint> -->
+  <!-- <disable_collisions link1="gripper" link2="link_6" reason="Never" /> -->
   <link name="camera"/>
   <joint name="camera_joint" type="fixed">

File: src/tm_description/xacro/macro.tm5x-900-nominal.urdf.xacro (robot description, xacro)
@@ -280,5 +280,5 @@
     <origin rpy="0.000000 0.000000 0.000000" xyz="0.000000 0.000000 0.000000" />
   </joint>
-  <link name="gripper">
+  <!-- <link name="gripper">
     <visual>
       <geometry>
@@ -300,5 +300,5 @@
     <origin rpy="-1.570795 0.000000 -1.570795" xyz="0 0 0.132"/>
   </joint>
-  <disable_collisions link1="gripper" link2="link_6" reason="Never" />
+  <disable_collisions link1="gripper" link2="link_6" reason="Never" /> -->
   <link name="camera">
   </link>

Commit message: 1. Add arduino_listener node 2. change laserTransform in moveit_demo to targetTransform 3. remove gripper description in order to rebuild new gripper description

File: src/tm_description/urdf/tm5-900.urdf (robot description, URDF)
Before this commit: robot tm5-900, 11 links, 10 joints
Links:
- removed link camera
Joints:
- removed joint camera_joint

File: src/tm_description/xacro/macro.tm5-900-nominal.urdf.xacro (robot description, xacro)
@@ -280,25 +280,4 @@
     <origin rpy="0.000000 0.000000 0.000000" xyz="0.000000 0.000000 0.000000" />
   </joint>
-  <!-- <link name="gripper">
-    <visual>
-      <geometry>
-        <mesh scale="0.001 0.001 0.001" filename="package://tm_description/meshes/gripper2023v1.stl"/>
-      </geometry>
-      <material name="Grey">
-        <color rgba="0.9 0.9 0.9 1.0"/>
-      </material>
-    </visual>
-    <collision>
-      <geometry>
-        <mesh scale="0.001 0.001 0.001" filename="package://tm_description/meshes/gripper2023v1.stl"/>
-      </geometry>
-    </collision>
-  </link> -->
-  <!-- <joint name="gripper_joint" type="fixed">
-    <parent link="${prefix}link_6"/>
-    <child link="gripper"/>
-    <origin rpy="-1.570795 0.000000 -1.570795" xyz="0 0 0.132"/>
-  </joint> -->
-  <!-- <disable_collisions link1="gripper" link2="link_6" reason="Never" /> -->
   <link name="camera"/>
   <joint name="camera_joint" type="fixed">

File: src/tm_description/xacro/macro.tm5x-900-nominal.urdf.xacro (robot description, xacro)
@@ -280,32 +280,4 @@
     <origin rpy="0.000000 0.000000 0.000000" xyz="0.000000 0.000000 0.000000" />
   </joint>
-  <!-- <link name="gripper">
-    <visual>
-      <geometry>
-        <mesh scale="0.001 0.001 0.001" filename="package://tm_description/meshes/gripper2023v1.stl"/>
-      </geometry>
-      <material name="Grey">
-        <color rgba="0.9 0.9 0.9 1.0"/>
-      </material>
-    </visual>
-    <collision>
-      <geometry>
-        <mesh scale="0.001 0.001 0.001" filename="package://tm_description/meshes/gripper2023v1.stl"/>
-      </geometry>
-    </collision>
-  </link>
-  <joint name="gripper_joint" type="fixed">
-    <parent link="${prefix}link_6"/>
-    <child link="gripper"/>
-    <origin rpy="-1.570795 0.000000 -1.570795" xyz="0 0 0.132"/>
-  </joint>
-  <disable_collisions link1="gripper" link2="link_6" reason="Never" /> -->
-  <link name="camera">
-  </link>
-  <joint name="camera_joint" type="fixed">
-    <parent link="${prefix}link_6"/>
-    <child link="camera"/>
-    <origin rpy="0.00000 0.000000 -1.570795" xyz="-0.0585 -0.0115 0.15995"/>
-  </joint>
 <!--LinkDescription-->
   </xacro:macro>
