Commit message: update gripper mesh

File: src/tm_description/xacro/macro.tm5-900-nominal.urdf.xacro (robot description, xacro)
@@ -283,5 +283,5 @@
     <visual>
       <geometry>
-        <mesh scale="0.001 0.001 0.001" filename="package://tm_description/meshes/Assembly1.stl"/>
+        <mesh scale="0.001 0.001 0.001" filename="package://tm_description/meshes/gripper2023v1.stl"/>
       </geometry>
       <material name="Grey">
@@ -291,5 +291,5 @@
     <collision>
       <geometry>
-        <mesh scale="0.001 0.001 0.001" filename="package://tm_description/meshes/Assembly1.stl"/>
+        <mesh scale="0.001 0.001 0.001" filename="package://tm_description/meshes/gripper2023v1.stl"/>
       </geometry>
     </collision>
@@ -298,5 +298,5 @@
     <parent link="${prefix}link_6"/>
     <child link="gripper"/>
-    <origin rpy="-1.570795 0.000000 -1.570795" xyz="0.0224 0.0001 0.1568"/>
+    <origin rpy="-1.570795 0.000000 -1.570795" xyz="0 0 0.132"/>
   </joint>
   <disable_collisions link1="gripper" link2="link_6" reason="Never" />

Commit message: add camera link

File: src/tm_description/xacro/macro.tm5-900-nominal.urdf.xacro (robot description, xacro)
@@ -301,4 +301,11 @@
   </joint>
   <disable_collisions link1="gripper" link2="link_6" reason="Never" />
+  <link name="camera">
+  </link>
+  <joint name="camera_joint" type="fixed">
+    <parent link="${prefix}link_6"/>
+    <child link="camera"/>
+    <origin rpy="0.00000 0.000000 -1.570795" xyz="-0.0585 -0.0115 0.15995"/>
+  </joint>
 <!--LinkDescription-->
   </xacro:macro>

Commit message: executiable gripper setting

File: src/tm_description/xacro/macro.tm5-900-nominal.urdf.xacro (robot description, xacro)
@@ -284,5 +284,22 @@
     <parent link="${prefix}link_6"/>
     <child link="camera"/>
-    <origin rpy="0.00000 0.000000 -1.570795" xyz="-0.0585 -0.0115 0.15995"/>
+    <origin rpy="0.00000 0.000000 -1.570795" xyz="-0.0585 0.000000 0.15995"/>
+  </joint>
+  <link name="gripper_link">
+    <visual>
+      <origin xyz="0 0 0" rpy="0.000000 0.000000 0.000000"/>
+      <!-- -1.570795 -->
+      <geometry>
+        <mesh scale="0.001 0.001 0.001" filename="package://tm_description/meshes/gripper.stl"/>
+      </geometry>
+      <material name="Grey">
+        <color rgba="0.9 0.9 0.9 1.0"/>
+      </material>
+    </visual>
+  </link>
+  <joint name="gripper_joint" type="fixed">
+    <parent link="${prefix}flange_link"/>
+    <child link="gripper_link"/>
+    <origin xyz="0 0 0.132" rpy="-1.570795 0.000000 -1.570795"/>
   </joint>
 <!--LinkDescription-->

Commit message: A new gripper model in meters

File: src/tm_description/xacro/macro.tm5-900-nominal.urdf.xacro (robot description, xacro)
@@ -291,5 +291,5 @@
       <!-- -1.570795 -->
       <geometry>
-        <mesh scale="0.001 0.001 0.001" filename="package://tm_description/meshes/gripper.stl"/>
+        <mesh filename="package://tm_description/meshes/gripper.stl"/>
       </geometry>
       <material name="Grey">
